File: Pyuta_Game_Adaptor/TOMY_Pyuuta_Game_Adaptor.kicad_sch (KiCad schematic)
At the start: 7 parts, among them J1 Tomy Pyūta I/O Port, J2 Tomy Pyūta Cartridge

Commit message: Updated from actual Game Adaptor
Connections:
- net V_{CC}: no longer J1.50 (V_{CC})
- net ~{MEMEN}: now reaches J1.21 (~{MEMEN})
- net ~{MEMEN}: now also J2.21 (~{CROM1})
- net ~{WE}: now reaches J1.31 (~{WE})
- net ~{WE}: now also J2.32 (~{WE})
- net ~{RESET}: now reaches J1.37 (~{RESET})
- net ~{RESET}: now also J2.4 (~{RESET})
- no-connect marks 27 -> 23
Changed lines of the file:
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@@
 	)
 	(junction
-		(at 113.03 114.3)
-		(diameter 0)
-		(color 0 0 0 0)
-	)
-	(junction
 		(at 129.54 62.23)
 		(diameter 0)
@@
 	)
 	(no_connect
-		(at 87.63 93.98)
+		(at 113.03 114.3)
 	)
 	(no_connect
-		(at 87.63 111.76)
+		(at 152.4 102.87)
 	)
 	(no_connect
@@
 	)
 	(no_connect
+		(at 115.57 138.43)
+	)
+	(no_connect
 		(at 113.03 111.76)
 	)
@@
 	)
 	(no_connect
-		(at 176.53 100.33)
+		(at 113.03 96.52)
 	)
 	(no_connect
-		(at 113.03 96.52)
+		(at 176.53 102.87)
 	)
 	(no_connect
@@
 	)
 	(no_connect
-		(at 176.53 64.77)
-	)
-	(no_connect
 		(at 87.63 106.68)
 	)
@@
 	)
 	(no_connect
-		(at 176.53 102.87)
+		(at 113.03 58.42)
 	)
 	(no_connect
-		(at 87.63 99.06)
+		(at 176.53 105.41)
 	)
 	(no_connect
-		(at 152.4 102.87)
+		(at 87.63 86.36)
 	)
 	(no_connect
-		(at 87.63 78.74)
+		(at 113.03 109.22)
 	)
 	(no_connect
-		(at 87.63 91.44)
+		(at 87.63 111.76)
 	)
 	(no_connect
@@
 	)
 	(no_connect
-		(at 113.03 58.42)
-	)
-	(no_connect
-		(at 87.63 86.36)
-	)
-	(no_connect
-		(at 113.03 109.22)
-	)
-	(no_connect
-		(at 176.53 105.41)
+		(at 87.63 93.98)
 	)
 	(no_connect
-		(at 152.4 87.63)
+		(at 113.03 99.06)
 	)
 	(no_connect
 		(at 87.63 104.14)
 	)
-	(no_connect
-		(at 113.03 99.06)
-	)
 	(wire
 		(pts
@@
 	(wire
 		(pts
-			(xy 129.54 85.09) (xy 129.54 114.3)
+			(xy 129.54 85.09) (xy 129.54 120.65)
 		)
 		(stroke
@@
 	(wire
 		(pts
-			(xy 113.03 120.65) (xy 113.03 114.3)
-		)
-		(stroke
-			(width 0)
-			(type default)
-		)
-	)
-	(wire
-		(pts
 			(xy 87.63 40.64) (xy 176.53 40.64)
 		)
@@
 	(wire
 		(pts
-			(xy 87.63 120.65) (xy 113.03 120.65)
+			(xy 87.63 120.65) (xy 129.54 120.65)
 		)
 		(stroke
@@
 		)
 	)
-	(wire
-		(pts
-			(xy 113.03 114.3) (xy 129.54 114.3)
-		)
-		(stroke
-			(width 0)
-			(type default)
-		)
-	)
 	(table
 		(column_count 3)
@@
 		)
 	)
+	(label "~{RESET}"
+		(at 176.53 64.77 0)
+		(effects
+			(font
+				(size 1.27 1.27)
+			)
+			(justify left bottom)
+		)
+	)
 	(label "GND"
 		(at 135.89 40.64 0)
@@
 		)
 	)
+	(label "~{MEMEN}"
+		(at 87.63 78.74 180)
+		(effects
+			(font
+				(size 1.27 1.27)
+			)
+			(justify right bottom)
+		)
+	)
 	(label "D_{1}"
 		(at 152.4 80.01 180)
@@
 		)
 	)
+	(label "~{WE}"
+		(at 176.53 100.33 0)
+		(effects
+			(font
+				(size 1.27 1.27)
+			)
+			(justify left bottom)
+		)
+	)
+	(label "~{WE}"
+		(at 87.63 91.44 180)
+		(effects
+			(font
+				(size 1.27 1.27)
+			)
+			(justify right bottom)
+		)
+	)
 	(label "D_{0}"
 		(at 87.63 73.66 180)
@@
 		)
 	)
+	(label "~{MEMEN}"
+		(at 152.4 87.63 180)
+		(effects
+			(font
+				(size 1.27 1.27)
+			)
+			(justify right bottom)
+		)
+	)
 	(label "SELEXM"
 		(at 176.53 67.31 0)
@@
 	)
 	(label "V_{CC}"
-		(at 118.11 114.3 0)
+		(at 91.44 120.65 0)
 		(effects
 			(font
@@
 		)
 	)
+	(label "~{RESET}"
+		(at 87.63 99.06 180)
+		(effects
+			(font
+				(size 1.27 1.27)
+			)
+			(justify right bottom)
+		)
+	)

Commit message: Initial design completed
Connections:
- no-connect marks 23 -> 22
Other:
- note removed: "NOTE! I am still pretty confused by the several dozen conflicting (in my mind) pinouts for the Western Tomy Tutor and the Japanese Pyūta. So please don't treat my design as error free and tested (24/Feb/2026)."
Changed lines of the file:
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@@
 		(rev "A")
 		(company "Brett Hallen")
-		(comment 3 "To enable a 32KB cartridge to work on the original Pyūta TP1000")
+		(comment 2 "Not required for ぴゅう太 Jr. (TP2001) or ぴゅう太 mk2 (TP1007)")
+		(comment 3 "To enable a 32KB cartridge to work on the original ぴゅう太 or Tutor (TP1000)")
 		(comment 4 "Homebrew version of the Game Adaptor (ゲーム アダプター)")
 	)
-	(text "NOTE!\nI am still pretty confused by the several dozen conflicting (in my mind) pinouts for the Western Tomy Tutor and the Japanese Pyūta.\nSo please don't treat my design as error free and tested (24/Feb/2026)."
-		(exclude_from_sim no)
-		(at 16.51 178.308 0)
-		(effects
-			(font
-				(size 1.27 1.27)
-			)
-			(justify left)
-		)
-	)
-	(text_box "Looking at the front of the cartridge:\nPin 1 = back right\nPin 2 = front right\nPin 35 = back left\nPin 36 = front left\n... I think"
+	(text_box "Looking at the front of the cartridge:\nPin 1 = back right\nPin 2 = front right\nPin 35 = back left\nPin 36 = front left"
 		(exclude_from_sim no)
 		(at 143.51 116.84 0)
-		(size 40.64 15.24)
+		(size 39.37 11.43)
 		(margins 0.9525 0.9525 0.9525 0.9525)
 		(stroke
@@
 	)
 	(no_connect
-		(at 115.57 138.43)
-	)
-	(no_connect
