File: Tomy_Pyuuta_Power_Supply/Tomy_Pyuuta_Power_Supply.kicad_sch (KiCad schematic)
At the start: 15 parts, among them J1 Power In (+12VDC), J2 Power Out, J3 Power LED, U1 +5V Regulator, U2 -5V Regulator

Commit message: Fixed 5V regulator pinout
Connections:
- net +5V: now also U1.3 (V_{OUT}); no longer U1.2 (V_{OUT})
- net GND: now also U1.2 (GND); no longer U1.3 (GND)

Commit message: Updated power connecters to JST
Parts:
- J1: footprint Connector_PinHeader_2.54mm:PinHeader_1x02_P2.54mm_Vertical -> Connector_JST:JST_NV_B02P-NV_1x02_P5.00mm_Vertical
- J2: footprint Connector_PinHeader_2.54mm:PinHeader_1x04_P2.54mm_Vertical -> Connector_JST:JST_NV_B04P-NV_1x04_P5.00mm_Vertical
- U1: footprint Package_TO_SOT_THT:TO-220-3_Vertical -> Package_TO_SOT_THT:TO-220-3_Horizontal_TabDown
Changed lines of the file:
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@@
 			)
 		)
-		(property "Footprint" "Connector_PinHeader_2.54mm:PinHeader_1x04_P2.54mm_Vertical"
+		(property "Footprint" "Connector_JST:JST_NV_B04P-NV_1x04_P5.00mm_Vertical"
 			(at 175.26 73.66 0)
 			(effects
@@
 			)
 		)
-		(property "Footprint" "Connector_PinHeader_2.54mm:PinHeader_1x02_P2.54mm_Vertical"
+		(property "Footprint" "Connector_JST:JST_NV_B02P-NV_1x02_P5.00mm_Vertical"
 			(at 69.85 74.676 0)
 			(effects
@@
 			)
 		)
-		(property "Footprint" "Package_TO_SOT_THT:TO-220-3_Vertical"
+		(property "Footprint" "Package_TO_SOT_THT:TO-220-3_Horizontal_TabDown"
 			(at 107.95 50.8 0)
 			(effects
